File: htr_reg/htr_reg.sch (EAGLE design)
At the start: 0 parts

Commit message: added a few more bits to the library, started assembling the schematic, brd file created.
Parts:
- added C1, C2, C3, C4, C5, C6: (no value), htr_reg_lib:CAP_SMD_0603
- added J1, J2, J3: XT30_EDGE, htr_reg_lib:XT30_EDGE
- added Q1, Q2: (no value), htr_reg_lib:MOSFET_N-CHANNEL_SOT23-3
- added R1, R2, R3: (no value), htr_reg_lib:RES_SMD0603
- added TC1, TC2: LMT85LPG, htr_reg_lib:LMT85LPG
- added TP1: (no value), htr_reg_lib:3296W
- added U1, U2: TLV3691_SC70-5, htr_reg_lib:TLV3691_SC70-5
- added U3: (no value), htr_reg_lib:78XX_VREG_B
