File: htr_reg/htr_reg.brd (EAGLE design)
At the start: 160 x 100 mm, 20 parts, among them J1 XT30_EDGE, J2 XT30_EDGE, J3 XT30_EDGE, U1 TLV3691_SC70-5, U2 TLV3691_SC70-5

Commit message: organized and connected the schematic
Parts:
- removed R3: (no value), htr_reg_lib:0603
- moved R1 23.0 mm to (-15.2, 41.9)
- moved R2 3.81 mm to (-19.1, 41.9)
Connections:
- new net 5V: C2.1, C3.1, C4.1, TC1.3, TC2.3, TP1.1, U1.5, U2.5, U3.2
- new net GND: C1.2, C2.2, C3.2, C4.2, C5.2, C6.2, J1.NEG, Q1.2, TC1.2, TC2.2, TP1.3, U1.2, U2.2, U3.1
- new net N$10: R1.1, TC1.1
- new net N$11: TP1.2, U1.1, U2.1
- new net N$3: Q2.1, U2.4
- new net N$4: Q1.1, U1.4
- new net N$5: J3.NEG, Q2.3
- new net N$6: J2.NEG, Q1.3
- new net N$7: C6.1, R2.2, U2.3
- new net N$8: R2.1, TC2.1
- new net N$9: C5.1, R1.2, U1.3
- new net V_IN: C1.1, J1.POS, J2.POS, J3.POS, U3.3
Changed lines of the file:
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@@
 <element name="Q1" library="htr_reg_lib" package="SOT23-3" value="" x="-24.13" y="35.56"/>
 <element name="Q2" library="htr_reg_lib" package="SOT23-3" value="" x="-27.94" y="35.56"/>
-<element name="R1" library="htr_reg_lib" package="0603" value="" x="-38.1" y="39.37"/>
-<element name="R2" library="htr_reg_lib" package="0603" value="" x="-15.24" y="41.91"/>
-<element name="R3" library="htr_reg_lib" package="0603" value="" x="-19.05" y="41.91"/>
+<element name="R1" library="htr_reg_lib" package="0603" value="" x="-15.24" y="41.91"/>
+<element name="R2" library="htr_reg_lib" package="0603" value="" x="-19.05" y="41.91"/>
 <element name="TC1" library="htr_reg_lib" package="TO-92" value="LMT85LPG" x="-35.56" y="25.4"/>
 <element name="TC2" library="htr_reg_lib" package="TO-92" value="LMT85LPG" x="-17.78" y="35.56"/>
@@
 </elements>
 <signals>
+<signal name="GND">
+<contactref element="TC1" pad="2"/>
+<contactref element="J1" pad="NEG"/>
+<contactref element="C2" pad="2"/>
+<contactref element="U3" pad="1"/>
+<contactref element="C1" pad="2"/>
+<contactref element="C3" pad="2"/>
+<contactref element="C4" pad="2"/>
+<contactref element="U2" pad="2"/>
+<contactref element="U1" pad="2"/>
+<contactref element="Q1" pad="2"/>
+<contactref element="C6" pad="2"/>
+<contactref element="TC2" pad="2"/>
+<contactref element="C5" pad="2"/>
+<contactref element="TP1" pad="3"/>
+<wire x1="-15.24" y1="8.89" x2="-32.98" y2="2.58" width="0" layer="19" extent="1-1"/>
+<wire x1="-35.56" y1="25.4" x2="-32.98" y2="2.58" width="0" layer="19" extent="1-1"/>
+<wire x1="-36.66" y1="34.29" x2="-35.56" y2="25.4" width="0" layer="19" extent="1-1"/>
+<wire x1="-40.47" y1="34.29" x2="-36.66" y2="34.29" width="0" layer="19" extent="1-1"/>
+<wire x1="-32.7" y1="34.56" x2="-36.66" y2="34.29" width="0" layer="19" extent="1-1"/>
+<wire x1="-33.44" y1="39.37" x2="-32.7" y2="34.56" width="0" layer="19" extent="1-1"/>
+<wire x1="-29.63" y1="39.37" x2="-33.44" y2="39.37" width="0" layer="19" extent="1-1"/>
+<wire x1="-25.82" y1="39.37" x2="-29.63" y2="39.37" width="0" layer="19" extent="1-1"/>
+<wire x1="-22.01" y1="39.37" x2="-25.82" y2="39.37" width="0" layer="19" extent="1-1"/>
+<wire x1="-18.2" y1="39.37" x2="-22.01" y2="39.37" width="0" layer="19" extent="1-1"/>
+<wire x1="-14.39" y1="39.37" x2="-18.2" y2="39.37" width="0" layer="19" extent="1-1"/>
+<wire x1="-17.78" y1="35.56" x2="-18.2" y2="39.37" width="0" layer="19" extent="1-1"/>
+<wire x1="-23.18" y1="34.56" x2="-22.01" y2="39.37" width="0" layer="19" extent="1-1"/>
+</signal>
+<signal name="5V">
+<contactref element="U3" pad="2"/>
+<contactref element="C2" pad="1"/>
+<contactref element="U1" pad="5"/>
+<contactref element="C3" pad="1"/>
+<contactref element="U2" pad="5"/>
+<contactref element="C4" pad="1"/>
+<contactref element="TC2" pad="3"/>
+<contactref element="TC1" pad="3"/>
+<contactref element="TP1" pad="1"/>
+<wire x1="-23.71" y1="39.37" x2="-19.9" y2="39.37" width="0" layer="19" extent="1-1"/>
+<wire x1="-27.52" y1="39.37" x2="-23.71" y2="39.37" width="0" layer="19" extent="1-1"/>
+<wire x1="-30.8" y1="34.56" x2="-27.52" y2="39.37" width="0" layer="19" extent="1-1"/>
+<wire x1="-34.46" y1="34.94" x2="-30.8" y2="34.56" width="0" layer="19" extent="1-1"/>
+<wire x1="-38.27" y1="34.94" x2="-34.46" y2="34.94" width="0" layer="19" extent="1-1"/>
+<wire x1="-15.24" y1="35.56" x2="-19.9" y2="39.37" width="0" layer="19" extent="1-1"/>
+<wire x1="-33.02" y1="25.4" x2="-30.8" y2="34.56" width="0" layer="19" extent="1-1"/>
+<wire x1="-15.24" y1="3.81" x2="-33.02" y2="25.4" width="0" layer="19" extent="1-1"/>
+</signal>
+<signal name="V_IN">
+<contactref element="U3" pad="3"/>
+<contactref element="J1" pad="POS"/>
+<contactref element="C1" pad="1"/>
+<contactref element="J2" pad="POS"/>
+<contactref element="J3" pad="POS"/>
+<wire x1="-27.9" y1="20.28" x2="-32.98" y2="7.58" width="0" layer="19" extent="1-1"/>
+<wire x1="-27.9" y1="30.44" x2="-27.9" y2="20.28" width="0" layer="19" extent="1-1"/>
+<wire x1="-31.75" y1="36.66" x2="-27.9" y2="30.44" width="0" layer="19" extent="1-1"/>
+<wire x1="-16.09" y1="39.37" x2="-27.9" y2="30.44" width="0" layer="19" extent="1-1"/>
+</signal>
+<signal name="N$3">
+<contactref element="U2" pad="4"/>
+<contactref element="Q2" pad="1"/>
+<wire x1="-28.89" y1="34.56" x2="-38.27" y2="33.64" width="0" layer="19" extent="1-1"/>
+</signal>
+<signal name="N$4">
+<contactref element="Q1" pad="1"/>
+<contactref element="U1" pad="4"/>
+<wire x1="-34.46" y1="33.64" x2="-25.08" y2="34.56" width="0" layer="19" extent="1-1"/>
+</signal>
+<signal name="N$5">
+<contactref element="Q2" pad="3"/>
+<contactref element="J3" pad="NEG"/>
+<wire x1="-27.9" y1="25.44" x2="-27.94" y2="36.66" width="0" layer="19" extent="1-1"/>
+</signal>
+<signal name="N$6">
+<contactref element="Q1" pad="3"/>
+<contactref element="J2" pad="NEG"/>
+<wire x1="-27.9" y1="15.28" x2="-24.13" y2="36.66" width="0" layer="19" extent="1-1"/>
+</signal>
+<signal name="N$7">
+<contactref element="U2" pad="3"/>
+<contactref element="C6" pad="1"/>
+<contactref element="R2" pad="2"/>
+<wire x1="-35.14" y1="39.37" x2="-18.2" y2="41.91" width="0" layer="19" extent="1-1"/>
+<wire x1="-40.47" y1="33.64" x2="-35.14" y2="39.37" width="0" layer="19" extent="1-1"/>
+</signal>
+<signal name="N$8">
+<contactref element="R2" pad="1"/>
+<contactref element="TC2" pad="1"/>
+<wire x1="-20.32" y1="35.56" x2="-19.9" y2="41.91" width="0" layer="19" extent="1-1"/>
+</signal>
+<signal name="N$9">
+<contactref element="U1" pad="3"/>
+<contactref element="C5" pad="1"/>
+<contactref element="R1" pad="2"/>
+<wire x1="-31.33" y1="39.37" x2="-14.39" y2="41.91" width="0" layer="19" extent="1-1"/>
+<wire x1="-36.66" y1="33.64" x2="-31.33" y2="39.37" width="0" layer="19" extent="1-1"/>
+</signal>
+<signal name="N$10">
+<contactref element="R1" pad="1"/>
+<contactref element="TC1" pad="1"/>
+<wire x1="-38.1" y1="25.4" x2="-16.09" y2="41.91" width="0" layer="19" extent="1-1"/>
+</signal>
+<signal name="N$11">
+<contactref element="U1" pad="1"/>
+<contactref element="U2" pad="1"/>
+<contactref element="TP1" pad="2"/>
+<wire x1="-36.66" y1="34.94" x2="-15.24" y2="6.35" width="0" layer="19" extent="1-1"/>
+<wire x1="-40.47" y1="34.94" x2="-36.66" y2="34.94" width="0" layer="19" extent="1-1"/>
+</signal>
 </signals>
 </board>

Commit message: Added and twiddled small bits of the lib. Routed traces on the board, possibly finished.
Parts:
- added D1, D2: (no value), htr_reg_lib:LED-0603
- added R3, R4: (no value), htr_reg_lib:0603
- TC1, TC2: value LMT85LPG -> LMT85.1"; device htr_reg_lib:TO-92 -> htr_reg_lib:1X03
- moved U2 59.5 mm to (12.7, 5.40)
- moved C6 59.2 mm to (12.7, 3.33)
- moved Q2 56.2 mm to (17.8, 2.86), turned to 270 degrees
- moved J3 55.7 mm to (25.4, 5.08)
- moved R2 51.3 mm to (12.7, 1.59), turned to 180 degrees
- moved J2 50.8 mm to (25.4, 17.8)
- moved C4 50.7 mm to (12.7, 7.46), turned to 180 degrees
- moved TC1 50.5 mm to (13.3, 12.7)
- moved U1 50.4 mm to (12.5, 19.2)
- moved U3 49.4 mm to (7.62, 5.71)
- moved C5 48.4 mm to (12.5, 17.1)
- moved Q1 46.0 mm to (17.8, 16.7), turned to 270 degrees
- moved C2 45.2 mm to (7.62, 2.86), turned to 180 degrees
- moved TC2 40.2 mm to (13.3, 10.2)
- moved C3 39.8 mm to (12.5, 21.3), turned to 180 degrees
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Connections:
- net N$10 renamed FB_A
- net N$11 renamed SET
- net N$8 renamed FB_B
- removed net N$3: Q2.1, U2.4
- new net N$2: D1.C, R3.1
- new net OUT_A: D1.A, Q1.1, U1.4
- new net OUT_B: D2.A, Q2.1, U2.4
- net 5V: now also TC1.2, TC2.2; no longer TC1.3, TC2.3
- net GND: now also Q2.2, R3.2, R4.2, TC1.3, TC2.3; no longer TC1.2, TC2.2
- net N$4: now also D2.C, R4.1; no longer Q1.1, U1.4
Routing:
- net 5V: track 0.00 -> 43.2 mm, vias 0 -> 2
- net SET: track 0.00 -> 18.3 mm
- net V_IN: track 0.00 -> 11.3 mm, vias 0 -> 27
- net FB_B: track 0.00 -> 10.0 mm, vias 0 -> 1
- net OUT_A: track 0.00 -> 5.12 mm
- net OUT_B: track 0.00 -> 4.96 mm
- net N$6: track 0.00 -> 4.60 mm
- net N$5: track 0.00 -> 4.13 mm
- net N$9: track 0.00 -> 3.18 mm
- net N$7: track 0.00 -> 3.18 mm
- net FB_A: track 0.00 -> 2.70 mm
- net N$2: track 0.00 -> 1.59 mm
- net N$4: track 0.00 -> 1.59 mm
- added copper zone on layer 1, net GND
- added copper zone on layer 16, net GND
- added copper zone on layer 16, net V_IN
Other:
- board size 160 x 100 mm -> 25.4 x 22.9 mm
